File: PCB/Aida_Plate_Mid_Inside/Aida_Plate_Mid_Inside.kicad_sch (KiCad schematic)
At the start: 5 parts

Commit message: プレート作成中
Parts:
- removed H1: GND from Mid, Lib_Local:MountingHole_M2_Through-hole_tap_THC-0.8-1.0-2_minimal, symbol Mechanical:MountingHole_Pad
- removed SW_RIGHT1: SW_Push, Lib_Local:Kailh_socket_ChocV2_for_Reverse, symbol Switch:SW_Push
- added H5: COL_4_to_Base, Lib_Local:MountingHole_2.2mm_M2_minimal, symbol Mechanical:MountingHole_Pad
- added SW_LEFT2, SW_LEFT3: SW_Push, Lib_Local:MX-Switch-Hole-with-narrow-frame, symbol Switch:SW_Push
- H2: value COL_4_from_Mid -> COL_3_from_Base; footprint Lib_Local:MountingHole_M2_Through-hole_tap_THC-0.8-1.0-2_minimal -> Lib_Local:MountingHole_2.2mm_M2_minimal
- H3: value COL_4_to_Base_via_Mid -> COL_3_to_Base; footprint Lib_Local:MountingHole_2.2mm_M2_Pad_minimal -> Lib_Local:MountingHole_2.2mm_M2_minimal
- SW_LEFT1: footprint Lib_Local:Kailh_socket_ChocV2_small_#2pad_for_Reverse_no_hole -> Lib_Local:MX-Switch-Hole-with-narrow-frame
Connections:
- net COL_4_from_Mid renamed COL_3_from_Base
- net COL_4_to_Base_via_Mid renamed COL_3_to_Base
- new net COL_4_from_Base: SW_LEFT2.1
- new net COL_4_to_Base: H5.1, SW_LEFT2.2
- new net COL_5_from_Base: SW_LEFT3.1
- new net COL_5_to_Base: SW_LEFT3.2
Other:
- note added: "Topのスイッチ出力は、 Midとは別にBaseへ伝達する。"
- moved on the sheet: H2, H3, SW_LEFT1
