File: PCB/Aida_Base/Aida_Base.kicad_pcb (KiCad board)
At the start: 2 copper layers, 3.1 x 4 mm, 224 parts, among them J1 AudioJack4, J10 Conn_01x03_Pin, J11 Conn_01x04_Pin, J12 Conn_01x04_Pin, J13 Conn_01x04_Pin, J14 Conn_01x04_Pin, J15 Conn_01x04_Pin, J16 Conn_01x04_Pin, J17 Conn_02x02_Odd_Even, J18 Conn_02x02_Odd_Even, J2 AudioJack4, J3 USB_C_Receptacle_L, J4 USB_C_Receptacle_R, J5 Conn_01x02_Pin, J6 Conn_01x02_Pin, J7 Conn_01x05_Pin, J8 Conn_01x05_Pin, J9 Conn_01x03_Pin, Q1 BSS138, Q2 BSS138, SW1 BOOT, SW2 BOOT, SW3 RESET, SW4 RESET, U1 NCP1117-3.3_SOT223, U2 NCP1117-3.3_SOT223, U3 RP2040_L, U4 RP2040_R, U5 W25Q128JVS, U6 W25Q128JVS, Y1 12MHz, Y2 12MHz

Commit message: 左手パーツ配置中。右手マトリクス修正
Parts:
- removed D6: D, Lib_Local:D_SOD-123_Emphasized_Direction_Line
- removed H10: MountingHole_Pad, Lib_Local:MountingHole_1.8-2.2mm_M2_Pad_minimal
- removed SW_A2, SW_B2, SW_C2, SW_CMD_L2, SW_CTL2, SW_D2, SW_E2, SW_F2, SW_OPT_L2, SW_S2, SW_SPC2, SW_V2, SW_W2, SW_X2, SW_Z2: SW_Push, Lib_Local:Kailh_socket_ChocV2
- removed SW_RE_L1: RotaryEncoder_Switch, Lib_Local:ChocV2_AND_RotaryEncoder_Alps_EC11K-Switch_Vertical_H20mm_NPTH_MP_minimal
- added ?: , clipboard:01c0b758-eab9-49d5-ba9f-7a87ce9b0684, F.Cu at (223.8, 57.1)
- added ?: , clipboard:01c0b758-eab9-49d5-ba9f-7a87ce9b0684, F.Cu at (71.4, 57.1)
- added H12: MountingHole_Pad, Lib_Local:MountingHole_1.8-2.2mm_M2_Pad_minimal, B.Cu at (-4.78, -62.4)
- added SW_-1: SW_Push, Lib_Local:Kailh_socket_ChocV2, B.Cu at (48.5, -108.6)
- added SW_/1: SW_Push, Lib_Local:Kailh_socket_ChocV2, B.Cu at (48.5, -91.7)
- added SW_<1: SW_Push, Lib_Local:Kailh_socket_ChocV2, B.Cu at (48.5, -74.9)
- added SW_>1: SW_Push, Lib_Local:Kailh_socket_ChocV2, B.Cu at (48.5, -58.0)
- added SW_BS1: SW_Push, Lib_Local:Kailh_socket_ChocV2, B.Cu at (48.5, -41.2)
- added SW_CMD_R1: SW_Push, Lib_Local:Kailh_socket_ChocV2, B.Cu at (48.5, -24.3)
- added SW_ENT1: SW_Push, Lib_Local:Kailh_socket_ChocV2, B.Cu at (30.4, -108.6)
- added SW_I1: SW_Push, Lib_Local:Kailh_socket_ChocV2, B.Cu at (30.4, -91.7)
- added SW_J1: SW_Push, Lib_Local:Kailh_socket_ChocV2, B.Cu at (30.4, -74.9)
- added SW_K1: SW_Push, Lib_Local:Kailh_socket_ChocV2, B.Cu at (30.4, -58.0)
- added SW_L1: SW_Push, Lib_Local:Kailh_socket_ChocV2, B.Cu at (30.4, -41.2)
- added SW_M1: SW_Push, Lib_Local:Kailh_socket_ChocV2, B.Cu at (30.4, -24.3)
- added SW_N1: SW_Push, Lib_Local:Kailh_socket_ChocV2, B.Cu at (12.2, -108.6)
- added SW_O1: SW_Push, Lib_Local:Kailh_socket_ChocV2, B.Cu at (12.2, -91.7)
- added SW_OPT_R1: SW_Push, Lib_Local:Kailh_socket_ChocV2, B.Cu at (12.2, -74.9)
- H1: value MountingHole_Pad -> COL_L_0_from_Mid_Outside
- H13: value MountingHole_Pad -> COL_L_4_from_Mid_Inside
- H15: value MountingHole_Pad -> COL_L_4_to_Mid_Inside
- H17: value MountingHole_Pad -> COL_L_5_from_Mid_Inside
- H19: value MountingHole_Pad -> COL_L_5_to_Mid_Inside
- H2: value MountingHole_Pad -> COL_L_3_from_Mid_Inside
- H3: value MountingHole_Pad -> COL_L_4_from_Top
- H7: value MountingHole_Pad -> COL_L_0_to_Mid_Outside
- H8: value MountingHole_Pad -> COL_L_3_to_Mid_Inside
- J11, J12, J15, J16: footprint Connector_PinHeader_2.54mm:PinHeader_1x04_P2.54mm_Vertical -> Connector_PinHeader_1.00mm:PinHeader_1x04_P1.00mm_Vertical
- J17, J18: footprint Connector_PinHeader_2.54mm:PinHeader_2x02_P2.54mm_Vertical -> Connector_PinHeader_2.00mm:PinHeader_2x02_P2.00mm_Vertical
- J5, J6: footprint Connector_PinHeader_2.54mm:PinHeader_1x02_P2.54mm_Vertical -> Connector_PinHeader_2.00mm:PinHeader_1x02_P2.00mm_Vertical
- J7, J8: footprint Connector_PinHeader_2.54mm:PinHeader_1x05_P2.54mm_Vertical -> Connector_PinHeader_1.00mm:PinHeader_1x05_P1.00mm_Vertical
- SW_A1, SW_B1, SW_C1, SW_CMD_L1, SW_CTL1, SW_D1, SW_E1, SW_F1, SW_OPT_L1, SW_S1, SW_SPC1, SW_V1, SW_W1, SW_X1, SW_Z1: moved to F.Cu
- moved C2 363.6 mm to (181.9, 39.3)
- moved R15 363.6 mm to (166.2, 32.1)
- moved R19 363.6 mm to (169.6, 39.3)
- moved R21 363.6 mm to (166.7, 36.9)
- moved D5 356.9 mm to (180.2, 26.2)
- moved H13 356.5 mm to (183.4, 71.4)
- moved C21 356.5 mm to (199.1, 48.8)
- moved C22 356.5 mm to (194.8, 48.8)
- moved C23 356.5 mm to (196.7, 53.6)
- moved C27 356.5 mm to (192.4, 58.8)
- moved C28 356.5 mm to (192.4, 60.7)
- moved H3 356.0 mm to (173.7, 25.8)
- moved LS1 355.4 mm to (166.7, 95.2)
- moved J17 346.7 mm to (159.5, 77.4)
- moved C1 346.3 mm to (164.3, 68.8), turned to -90 degrees
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Connections:
- H14 pad 1: Net-(D22-A) -> Net-(D18-A)
- H18 pad 1: Net-(D34-A) -> Net-(D29-A)
- H4 pad 1: Net-(D7-A) -> Net-(D8-A)
- H5 pad 1: Net-(D10-A) -> Net-(D9-A)
- H6 pad 1: Net-(D11-A) -> Net-(D12-A)
- SW_RE_L2 pad S2: Net-(D12-A) -> Net-(D7-A)
Routing:
- added copper zone on B.Cu, net GND_L
- added copper zone on F.Cu, net GND_L
Other:
- board size 3.1 x 4 mm -> 271.5 x 81 mm

Commit message: 左手パーツ配置中。ネジ位置で悩み中。
Parts:
- moved H_btm_L1 61.1 mm to (49.4, 93.5)
- moved C33 54.6 mm to (180.3, 73.8)
- moved C32 51.7 mm to (180.3, 69.7)
- moved C34 47.7 mm to (180.3, 78.0)
- moved H2 45.7 mm to (150.0, 66.7)
- moved D4 44.2 mm to (150.2, 70.8)
- moved R16 43.5 mm to (173.8, 66.1)
- moved H19 30.5 mm to (159.5, 85.7)
- moved D5 30.1 mm to (166.6, 53.0)
- moved H_mid_L2 27.0 mm to (88.1, 45.8)
- moved D1 24.4 mm to (74.4, 64.3)
- moved H15 23.0 mm to (166.1, 66.7)
- moved H7 22.7 mm to (71.4, 47.6)
- moved D17 22.2 mm to (170.3, 82.2)
- moved H3 21.2 mm to (166.7, 45.8)
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Other:
- board size 271.5 x 81 mm -> 271.5 x 185.1 mm
- board text added: "直径=3.0mm"
- board text added: "直径=3.5mm"
- board text added: "直径=4.0mm"

Commit message: 左手パーツ配置中。ネジ位置ほぼ確定。MCUまわり配置中。
Parts:
- added L4: SK6812MINI-E, locallib:YS-SK6812MINI-E_middle_hole_with_small_pad, B.Cu at (194.1, 70.8)
- added L5: SK6812MINI-E, locallib:YS-SK6812MINI-E_middle_hole_with_small_pad, B.Cu at (194.1, 75.6)
- added L6: SK6812MINI-E, locallib:YS-SK6812MINI-E_middle_hole_with_small_pad, B.Cu at (194.1, 80.4)
- H1, H13, H15, H17, H19, H2, H3, H7, H8, H_mid_L1, H_mid_L2: footprint Lib_Local:MountingHole_1.8-2.2mm_M2_Pad_minimal -> Lib_Local:MountingHole_M2_Through-hole_tap_THC-0.8-2.0-2_minimal; moved to F.Cu
- H11, H12, H14, H16, H18, H20, H4, H5, H6, H_mid_R1, H_mid_R2: footprint Lib_Local:MountingHole_1.8-2.2mm_M2_Pad_minimal -> Lib_Local:MountingHole_M2_Through-hole_tap_THC-0.8-2.0-2_minimal
- H_btm_L1, H_btm_L2, H_btm_L3, H_btm_L4, H_btm_L5, H_btm_L6: footprint Lib_Local:MountingHole_2.2mm_M2_No_Cu -> Lib_Local:MountingHole_M2_Through-hole_tap_THC-0.8-1.0-2_minimal; moved to F.Cu
- H_btm_R1, H_btm_R2, H_btm_R3, H_btm_R4, H_btm_R5, H_btm_R6: footprint Lib_Local:MountingHole_2.2mm_M2_No_Cu -> Lib_Local:MountingHole_M2_Through-hole_tap_THC-0.8-1.0-2_minimal
- SW_-1, SW_/1, SW_<1, SW_>1, SW_BS1, SW_CMD_R1, SW_ENT1, SW_I1, SW_J1, SW_K1, SW_L1, SW_M1, SW_N1, SW_O1, SW_OPT_R1: moved to F.Cu
- moved H_btm_L6 119.3 mm to (156.0, 123.2)
- moved SW_CMD_R1 100.1 mm to (62.2, -123.5)
- moved SW_M1 100.1 mm to (44.1, -123.5)
- moved H_btm_L4 71.8 mm to (109.5, 85.7)
- moved SW_-1 70.6 mm to (62.2, -39.3)
- moved SW_ENT1 70.6 mm to (44.1, -39.3)
- moved SW_N1 70.6 mm to (25.9, -39.3)
- moved SW_BS1 66.9 mm to (62.2, -106.7)
- moved SW_L1 66.9 mm to (44.1, -106.7)
- moved H_btm_L5 62.7 mm to (95.8, 123.2)
- moved C28 48.3 mm to (145.3, 50.0)
- moved C27 47.7 mm to (145.3, 51.2)
- moved C2 44.1 mm to (140.3, 53.6)
- moved H_btm_L3 43.9 mm to (62.5, 85.7)
- moved SW_/1 38.1 mm to (62.2, -56.1)
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Other:
- outline, holes or cut-outs redrawn
- board text added: "Place Reset & Boot SW besides Regulator"
- board text added: "SandyLP LEDs"

Commit message: 基板4枚、位置決め完了。
Parts:
- removed C21, C24: 2.2uF, Capacitor_SMD:C_0402_1005Metric
- removed H_btm_L1, H_btm_L2, H_btm_R1, H_btm_R2: MountingHole, Lib_Local:MountingHole_M2_Through-hole_tap_THC-0.8-1.0-2_minimal
- removed U1, U2: NCP1117-3.3_SOT223, Package_TO_SOT_SMD:SOT-223-3_TabPin2
- added R27: 27, Resistor_SMD:R_0402_1005Metric, B.Cu at (116.1, 41.1)
- added R28: 27, Resistor_SMD:R_0402_1005Metric, B.Cu at (-81.5, -25.8)
- added R29: 27, Resistor_SMD:R_0402_1005Metric, B.Cu at (116.1, 39.9)
- added R30: 27, Resistor_SMD:R_0402_1005Metric, B.Cu at (-75.5, -25.8)
- added U7: AP2112K-3.3, Package_TO_SOT_SMD:SOT-23-5, B.Cu at (105.4, 45.2)
- added U8: AP2112K-3.3, Package_TO_SOT_SMD:SOT-23-5, B.Cu at (-66.1, -2.03)
- C27, C28, C29, C30: value 2.2uF -> 1u
- J1: footprint Connector_Audio:Jack_3.5mm_PJ320E_Horizontal -> Lib_Local:TRRS-PJ-320A; moved to F.Cu
- J2: footprint Connector_Audio:Jack_3.5mm_PJ320E_Horizontal -> Lib_Local:TRRS-PJ-320A
- U3, U4: footprint Package_DFN_QFN:QFN-56-1EP_7x7mm_P0.4mm_EP3.2x3.2mm -> Lib_Local:RP2040-QFN-56
- moved C1 83.0 mm to (100.0, 46.2)
- moved C23 78.2 mm to (118.5, 54.8), turned to -90 degrees
- moved C10 75.1 mm to (112.7, 44.1)
- moved C9 74.1 mm to (113.7, 42.9)
- moved C5 73.8 mm to (114.3, 48.2)
- moved C12 71.7 mm to (117.9, 36.9), turned to 90 degrees
- moved J9 71.7 mm to (109.7, 61.9), turned to 90 degrees
- moved C11 70.1 mm to (119.1, 36.9), turned to 90 degrees
- moved C6 69.2 mm to (119.7, 54.8), turned to -90 degrees
- moved C22 69.1 mm to (126.2, 39.9), turned to 0 degrees
- moved C7 60.4 mm to (127.4, 48.2), turned to 0 degrees
- moved C8 60.3 mm to (127.4, 44.6), turned to 0 degrees
- moved F1 40.7 mm to (48.8, 47.6)
- moved C32 40.6 mm to (141.1, 58.9), turned to 90 degrees
- moved J7 40.5 mm to (130.4, 74.0), turned to 180 degrees
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Connections:
- L4 pad 2: Net-(L4-DOUT) -> (no net)
- L4 pad 4: LED_D_5V_CONNECTION -> (no net)
- L5 pad 2: Net-(L5-DOUT) -> (no net)
- L5 pad 4: Net-(L4-DOUT) -> (no net)
- L6 pad 2: unconnected-(L6-DOUT-Pad2) -> (no net)
- L6 pad 4: Net-(L5-DOUT) -> (no net)
- U3 pad 46: D-_L -> Net-(U3-USB_DM)
- U3 pad 47: D+_L -> Net-(U3-USB_DP)
- U4 pad 46: D-_R -> Net-(U4-USB_DM)
- U4 pad 47: D+_R -> Net-(U4-USB_DP)
Routing:
- net QSPI_SD2_L: track 0.00 -> 1.58 mm
- added copper zone on B.Cu, net +1V1_L
- added copper zone on B.Cu, net +3V3_L
Other:
- board size 271.5 x 185.1 mm -> 300 x 195.3 mm
- board text added: "Mid PCB-inside outline"
- board text added: "PCB Mid-Outside outline"
- board text added: "Top PCB outline"
- board text removed: "Place Reset & Boot SW besides Regulator"

Commit message: プレート作成中
Parts:
- moved H_mid_L1 1.19 mm to (123.8, 36.3)
- moved H15 1.19 mm to (147.6, 52.4)
Other:
- board text added: "Mid PCB outline"
- board text added: "中央のネジを1/32u上へ移動したい。 Base用プレートで、 下のスイッチにちょっとかぶり気味になっている。"
- board text removed: "Mid PCB-inside outline"

Commit message: プレート類調整中。LED位置検討中。
Parts:
- moved R16 4.76 mm to (135.7, 57.2)
- moved C31 4.76 mm to (135.1, 58.9)
- moved C32 4.76 mm to (136.3, 58.9)
- moved C33 4.76 mm to (136.3, 63.7)
- moved C34 4.76 mm to (136.3, 68.5)
- moved L1 3.04 mm to (142.9, 59.5)
- moved L2 3.04 mm to (142.9, 64.3)
- moved L3 3.04 mm to (142.9, 69.1)
Other:
- board text added: "LED位置検討中"
- board text removed: "中央のネジを1/32u上へ移動したい。 Base用プレートで、 下のスイッチにちょっとかぶり気味になっている。"
Changed lines of the file:
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@@
 	(generator_version "9.0")
 	(general
-		(thickness 1.6)
+		(thickness 1.2)
 		(legacy_teardrops no)
 	)
@@
 	)
 	(setup
+		(stackup
+			(layer "F.SilkS"
+				(type "Top Silk Screen")
+			)
+			(layer "F.Paste"
+				(type "Top Solder Paste")
+			)
+			(layer "F.Mask"
+				(type "Top Solder Mask")
+				(thickness 0.01)
+			)
+			(layer "F.Cu"
+				(type "copper")
+				(thickness 0.035)
+			)
+			(layer "dielectric 1"
+				(type "core")
+				(thickness 1.11)
+				(material "FR4")
+				(epsilon_r 4.5)
+				(loss_tangent 0.02)
+			)
+			(layer "B.Cu"
+				(type "copper")
+				(thickness 0.035)
+			)
+			(layer "B.Mask"
+				(type "Bottom Solder Mask")
+				(thickness 0.01)
+			)
+			(layer "B.Paste"
+				(type "Bottom Solder Paste")
+			)
+			(layer "B.SilkS"
+				(type "Bottom Silk Screen")
+			)
+			(copper_finish "None")
+			(dielectric_constraints no)
+		)
 		(pad_to_mask_clearance 0)
 		(allow_soldermask_bridges_in_footprints no)
@@
 	(footprint "Capacitor_SMD:C_0402_1005Metric"
 		(layer "B.Cu")
-		(at 139.898559 58.935967 90)
+		(at 135.135937 58.935967 90)
 		(descr "Capacitor SMD 0402 (1005 Metric), square (rectangular) end terminal, IPC-7351 nominal, (Body size source: IPC-SM-782 page 76, https://www.pcb-3d.com/wordpress/wp-content/uploads/ipc-sm-782a_amendment_1_and_2.pdf), generated with kicad-footprint-generator")
 		(tags "capacitor")
@@
 	(footprint "Lib_Local:YS-SK6812MINI-E_middle_hole_with_small_pad"
 		(layer "B.Cu")
-		(at 145.851665 63.698471 180)
+		(at 142.875 64.29375 180)
 		(property "Reference" "L2"
 			(at 0 -2.8 0)
@@
 	(footprint "Capacitor_SMD:C_0402_1005Metric"
 		(layer "B.Cu")
-		(at 141.089185 63.698471 90)
+		(at 136.326563 63.698471 90)
 		(descr "Capacitor SMD 0402 (1005 Metric), square (rectangular) end terminal, IPC-7351 nominal, (Body size source: IPC-SM-782 page 76, https://www.pcb-3d.com/wordpress/wp-content/uploads/ipc-sm-782a_amendment_1_and_2.pdf), generated with kicad-footprint-generator")
 		(tags "capacitor")
@@
 	(footprint "Resistor_SMD:R_0402_1005Metric"
 		(layer "B.Cu")
-		(at 140.493872 57.150028)
+		(at 135.73125 57.150028)
 		(descr "Resistor SMD 0402 (1005 Metric), square (rectangular) end terminal, IPC-7351 nominal, (Body size source: IPC-SM-782 page 72, https://www.pcb-3d.com/wordpress/wp-content/uploads/ipc-sm-782a_amendment_1_and_2.pdf), generated with kicad-footprint-generator")
 		(tags "resistor")
@@
 	(footprint "Capacitor_SMD:C_0402_1005Metric"
 		(layer "B.Cu")
-		(at 141.089185 68.460975 90)
+		(at 136.326563 68.460975 90)
 		(descr "Capacitor SMD 0402 (1005 Metric), square (rectangular) end terminal, IPC-7351 nominal, (Body size source: IPC-SM-782 page 76, https://www.pcb-3d.com/wordpress/wp-content/uploads/ipc-sm-782a_amendment_1_and_2.pdf), generated with kicad-footprint-generator")
 		(tags "capacitor")
@@
 	(footprint "Lib_Local:YS-SK6812MINI-E_middle_hole_with_small_pad"
 		(layer "B.Cu")
-		(at 145.851665 58.935967 180)
+		(at 142.875 59.531246 180)
 		(property "Reference" "L1"
 			(at 0 -2.8 0)
@@
 	(footprint "Capacitor_SMD:C_0402_1005Metric"
 		(layer "B.Cu")
-		(at 141.089185 58.935967 90)
+		(at 136.326563 58.935967 90)
 		(descr "Capacitor SMD 0402 (1005 Metric), square (rectangular) end terminal, IPC-7351 nominal, (Body size source: IPC-SM-782 page 76, https://www.pcb-3d.com/wordpress/wp-content/uploads/ipc-sm-782a_amendment_1_and_2.pdf), generated with kicad-footprint-generator")
 		(tags "capacitor")
@@
 	(footprint "Lib_Local:YS-SK6812MINI-E_middle_hole_with_small_pad"
 		(layer "B.Cu")
-		(at 145.851665 68.460975 180)
+		(at 142.875 69.056254 180)
 		(property "Reference" "L3"
 			(at 0 -2.8 0)
@@
 		)
 	)
-	(gr_text "中央のネジを1/32u上へ移動したい。\nBase用プレートで、\n下のスイッチにちょっとかぶり気味になっている。"
-		(at 88.701617 127.396962 0)
-		(layer "Eco2.User")
-		(effects
-			(font
-				(size 1.5 1.5)
-				(thickness 0.1875)
-			)
-			(justify left bottom)
-		)
-	)
 	(gr_text "直径=3.5mm"
 		(at 163.103992 42.267476 0)
@@
 		)
 	)
+	(gr_text "LED位置検討中"
+		(at 153.590625 64.29375 0)
+		(layer "Eco2.User")
+		(effects
+			(font
+				(size 2 2)
+				(thickness 0.25)
+			)
+			(justify left bottom)
+		)
+	)
 	(segment
 		(start 132.715 44.866575)
@@
 		)
 	)
+	(group ""
+		(members "15758f67-a113-4c90-8a75-4c840e81cfe7" "75793e4a-507a-4bda-ba5d-69b7a00169f9"
+			"d2e91539-892f-4984-88d4-b71cd9922127"
+		)
+	)

Commit message: LED位置、とりあえず決定。
Parts:
- removed the L4 at (194.7, 69.1)
- removed the L5 at (194.7, 73.8)
- removed the L6 at (194.7, 78.6)
- moved ? 194.1 mm to (53.9, 150.8)
Other:
- board size 300 x 195.3 mm -> 119.7 x 83.3 mm
- board text removed: "LED位置検討中"
- board text removed: "SandyLP LEDs"
