File: PCB/Aida_Base/Aida_Base.kicad_pcb (KiCad board)
At the start: 2 copper layers, 119.7 x 83.3 mm, 222 parts, among them J1 AudioJack4, J10 Conn_01x03_Pin, J11 Conn_01x04_Pin, J12 Conn_01x04_Pin, J13 Conn_01x04_Pin, J14 Conn_01x04_Pin, J15 Conn_01x04_Pin, J16 Conn_01x04_Pin, J17 Conn_02x02_Odd_Even, J18 Conn_02x02_Odd_Even, J2 AudioJack4, J3 USB_C_Receptacle_L, J4 USB_C_Receptacle_R, J5 Conn_01x02_Pin, J6 Conn_01x02_Pin, J7 Conn_01x05_Pin, J8 Conn_01x05_Pin, J9 Conn_01x03_Pin, Q1 BSS138, Q2 BSS138, SW1 BOOT, SW2 BOOT, SW3 RESET, SW4 RESET, U3 RP2040_L, U4 RP2040_R, U5 W25Q128JVS, U6 W25Q128JVS, U7 AP2112K-3.3, U8 AP2112K-3.3, Y1 12MHz, Y2 12MHz

Commit message: 右手パーツ配置中
Parts:
- removed SW_RE_L2: RotaryEncoder_Switch, Lib_Local:ChocV2_AND_RotaryEncoder_Alps_EC11K-Switch_Vertical_H20mm_NPTH_MP_minimal
- C1, C2, C3, C4: footprint Capacitor_SMD:C_0805_2012Metric -> Capacitor_SMD:C_0402_1005Metric
- H11: value MountingHole_Pad -> COL_R_3_to_Mid; moved to F.Cu
- H12: value MountingHole_Pad -> COL_R_0_to_Mid_Outside; moved to F.Cu
- H14: value MountingHole_Pad -> COL_R_4_from_Mid; moved to F.Cu
- H16: value MountingHole_Pad -> COL_R_4_to_Mid/Top; moved to F.Cu
- H18: value MountingHole_Pad -> COL_R_5_from_Mid; moved to F.Cu
- H20: value MountingHole_Pad -> COL_R_5_to_Mid; moved to F.Cu
- H4: value MountingHole_Pad -> COL_R_4_from_Top; moved to F.Cu
- H5: value MountingHole_Pad -> COL_R_3_from_Mid; moved to F.Cu
- H6: value MountingHole_Pad -> COL_R_0_from_Mid_Outside; moved to F.Cu
- H_btm_R3, H_btm_R4, H_btm_R5, H_btm_R6: moved to F.Cu
- H_mid_L1, H_mid_L2: footprint Lib_Local:MountingHole_M2_Through-hole_tap_THC-0.8-2.0-2_minimal -> Lib_Local:MountingHole_M2_Through-hole_tap_THC-0.8-1.0-2_minimal
- H_mid_R1, H_mid_R2: footprint Lib_Local:MountingHole_M2_Through-hole_tap_THC-0.8-2.0-2_minimal -> Lib_Local:MountingHole_M2_Through-hole_tap_THC-0.8-1.0-2_minimal; moved to F.Cu
- J1, J2: footprint Lib_Local:TRRS-PJ-320A -> Lib_Local:TRRS-PJ-320A_PinNameChanged
- J5, J6: footprint Connector_PinHeader_2.00mm:PinHeader_1x02_P2.00mm_Vertical -> Connector_PinHeader_2.00mm:PinHeader_1x03_P2.00mm_Vertical
- moved C13 423.4 mm to (351.3, 86.3)
- moved C14 423.4 mm to (342.7, 83.9)
- moved C15 423.4 mm to (346.5, 83.9)
- moved C16 423.4 mm to (344.1, 79.2)
- moved C17 423.4 mm to (348.9, 79.2)
- moved C18 423.4 mm to (304.1, -40.3)
- moved C19 423.4 mm to (304.1, -38.3)
- moved C20 423.4 mm to (304.1, -36.3)
- moved C25 423.4 mm to (301.2, -44.2)
- moved C26 423.4 mm to (301.2, -42.2)
- moved C29 423.4 mm to (301.2, -36.3)
- moved C3 423.4 mm to (295.8, 21.5)
- moved C30 423.4 mm to (301.2, -34.4)
- moved C35 423.4 mm to (298.4, -42.2)
- moved C36 423.4 mm to (298.4, -40.3)
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Connections:
- H_btm_L3 pad 1: (no net) -> GND_L
- H_btm_L4 pad 1: (no net) -> GND_L
- H_btm_L5 pad 1: (no net) -> GND_L
- H_btm_L6 pad 1: (no net) -> GND_L
- H_btm_R3 pad 1: (no net) -> GND_R
- H_btm_R4 pad 1: (no net) -> GND_R
- H_btm_R5 pad 1: (no net) -> GND_R
- H_btm_R6 pad 1: (no net) -> GND_R
- J3 pad A8: unconnected-(J3-SBU1-PadA8) -> (no net)
- J3 pad B8: unconnected-(J3-SBU2-PadB8) -> (no net)
- J4 pad A8: unconnected-(J4-SBU1-PadA8) -> (no net)
- J4 pad B8: unconnected-(J4-SBU2-PadB8) -> (no net)
- J5 pad 2: +3V3_L -> GND_L
- J6 pad 2: +3V3_R -> GND_R
Routing:
- net D-_L: track 0.00 -> 64.1 mm
- net D+_L: track 0.00 -> 63.6 mm
- net +5V_L: track 0.00 -> 47.5 mm
- net +3V3_L: track 0.00 -> 34.4 mm
- net +1V1_L: track 0.00 -> 22.5 mm, vias 0 -> 4
- net QSPI_SD3_L: track 0.00 -> 20.5 mm
- net QSPI_SS_L: track 0.00 -> 18.7 mm
- net QSPI_SCLK_L: track 0.00 -> 18.4 mm
- net QSPI_SD1_L: track 0.00 -> 18.3 mm
- net QSPI_SD2_L: track 1.58 -> 17.5 mm
- net QSPI_SD0_L: track 0.00 -> 15.1 mm
- net VBUS_L: track 0.00 -> 9.25 mm
- net Net-(U3-USB_DP): track 0.00 -> 5.41 mm
- net Net-(U3-USB_DM): track 0.00 -> 4.25 mm
- net Net-(U3-XOUT): track 0.00 -> 3.49 mm
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Other:
- board size 119.7 x 83.3 mm -> 242.9 x 83.3 mm
- board text added: "中央ネジ穴は 下のスイッチに干渉しないよう 1/32u上へオフセット"

Commit message: マトリクス行列のテストポイント追加
Parts:
- added J19: Conn_01x04_Pin, Connector_PinHeader_2.00mm:PinHeader_1x04_P2.00mm_Vertical, B.Cu at (55.9, 76.2)
- added J20: Conn_01x06_Pin, Connector_PinHeader_2.00mm:PinHeader_1x06_P2.00mm_Vertical, B.Cu at (71.0, 76.2)
- added J21: Conn_01x06_Pin, Connector_PinHeader_2.00mm:PinHeader_1x06_P2.00mm_Vertical, B.Cu at (297.9, 102.8)
- added J22: Conn_01x04_Pin, Connector_PinHeader_2.00mm:PinHeader_1x04_P2.00mm_Vertical, B.Cu at (306.0, 102.8)
- J2: moved to F.Cu
- moved J2 219.5 mm to (158.4, 35.7), turned to 0 degrees
- moved R4 152.9 mm to (158.4, 42.9)

Commit message: 左手側配線中
Routing:
- net COL_L_4: track 0.00 -> 171.1 mm, vias 0 -> 7
- net COL_L_0: track 0.00 -> 168.9 mm, vias 0 -> 4
- net ROW_L_3: track 0.00 -> 164.7 mm, vias 0 -> 3
- net ROW_L_2: track 0.00 -> 154.3 mm, vias 0 -> 3
- net ROW_L_1: track 0.00 -> 146.2 mm, vias 0 -> 3
- net COL_L_2: track 0.00 -> 133.3 mm, vias 0 -> 6
- net COL_L_5: track 0.00 -> 126.9 mm, vias 0 -> 3
- net COL_L_3: track 0.00 -> 120.2 mm, vias 0 -> 5
- net COL_L_1: track 0.00 -> 116.6 mm, vias 0 -> 4
- net ROW_L_0: track 0.00 -> 82.4 mm, vias 0 -> 1
- net +5V_L: track 47.5 -> 120.3 mm
- net Net-(D17-A): track 0.00 -> 50.4 mm
- net GPIO00_L: track 0.00 -> 47.8 mm, vias 0 -> 1
- net LED_5V_L: track 0.00 -> 47.6 mm
- net GPIO01_L: track 0.00 -> 47.1 mm, vias 0 -> 1
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
Commit message: 左手側配線。ほぼ完了。
Parts:
- added J23: Conn_01x02_Pin, Connector_PinHeader_2.00mm:PinHeader_1x02_P2.00mm_Vertical, B.Cu at (91.6, 61.8)
- added J24: Conn_01x02_Pin, Connector_PinHeader_2.00mm:PinHeader_1x02_P2.00mm_Vertical, F.Cu at (155.8, 26.6)
- added TP1: TestPoint, Connector_PinHeader_2.00mm:PinHeader_1x01_P2.00mm_Vertical, B.Cu at (144.7, 42.0)
- added TP2: TestPoint, Connector_PinHeader_2.00mm:PinHeader_1x01_P2.00mm_Vertical, F.Cu at (156.0, 21.4)
- moved R3 1.04 mm to (147.0, 42.0), turned to -90 degrees
Routing:
- net +3V3_L: track 75.6 -> 213.9 mm, vias 0 -> 9
- net GPIO22_L: track 0.00 -> 83.2 mm, vias 0 -> 2
- net GPIO23_L: track 0.00 -> 82.8 mm, vias 0 -> 2
- net GPIO24_L: track 0.00 -> 81.9 mm, vias 0 -> 2
- net SDA_L: track 2.63 -> 83.9 mm, vias 0 -> 2
- net GPIO25_L: track 0.00 -> 80.9 mm, vias 0 -> 2
- net SCL_L: track 2.56 -> 81.9 mm, vias 0 -> 2
- net SWCLK_L: track 0.00 -> 76.7 mm, vias 0 -> 2
- net SWDIO_L: track 0.00 -> 73.0 mm, vias 0 -> 2
- net RESET_L: track 4.15 -> 77.1 mm, vias 0 -> 3
- net ROW_L_0: track 82.4 -> 146.7 mm, vias 1 -> 3
- net GPIO26_L: track 0.00 -> 61.9 mm, vias 0 -> 2
- net GPIO27_L: track 0.00 -> 59.1 mm, vias 0 -> 2
- net GPIO28_L: track 0.00 -> 58.3 mm, vias 0 -> 2
- net GPIO29_L: track 0.00 -> 56.3 mm, vias 0 -> 2
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
Commit message: ボトムプレートの穴あけ用に、左手側パーツ配置調整。
Parts:
- R23, R24, R25, R26: footprint Resistor_SMD:R_0402_1005Metric -> Resistor_SMD:R_0603_1608Metric_Pad0.98x0.95mm_HandSolder
- moved R9 21.6 mm to (134.5, 92.0)
- moved J17 18.8 mm to (106.0, 84.8)
- moved D45 16.6 mm to (125.0, 88.1)
- moved D17 12.1 mm to (115.5, 66.7)
- moved D28 12.1 mm to (125.0, 85.7)
- moved J23 7.14 mm to (96.8, 66.7)
- moved J20 5.64 mm to (74.0, 81.0)
- moved J19 5.10 mm to (57.7, 81.0)
- moved JP1 3.57 mm to (125.0, 64.2)
- moved R1 3.57 mm to (125.0, 67.2), turned to 0 degrees
- moved STLED1 3.57 mm to (125.0, 69.1), turned to 0 degrees
- moved SW1 3.57 mm to (129.8, 64.3)
- moved SW3 3.57 mm to (129.8, 68.5)
- moved J11 3.17 mm to (130.4, 94.1)
- moved R23 1.81 mm to (141.1, 92.0)
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Connections:
- net D+_L renamed D_L+
- net D+_R renamed D_R+
- net D-_L renamed D_L-
- net D-_R renamed D_R-
Routing:
- net BUZZ_L: track 32.8 -> 66.2 mm
- net USB_BOOT_L: track 50.9 -> 72.1 mm
- net GND_L: track 25.2 -> 44.5 mm, vias 5 -> 18
- net +5V_L: track 120.0 -> 136.4 mm, vias 0 -> 3
- net Net-(D28-A): track 41.0 -> 25.5 mm
- net RESET_L: track 77.1 -> 62.7 mm
- net Net-(LS1-Pad1): track 20.1 -> 6.19 mm, vias 2 -> 0
- net ROW_L_1: track 147.4 -> 160.9 mm
- net Net-(D17-A): track 50.5 -> 38.6 mm
- net COL_L_4: track 145.2 -> 136.3 mm, vias 6 -> 5
- net ROW_L_2: track 156.9 -> 150.8 mm, vias 3 -> 2
- net ROW_L_0: track 146.7 -> 152.2 mm
- net ROW_L_3: track 164.8 -> 159.8 mm
- net ENC_L_B: track 36.8 -> 32.7 mm
- net ENC_L_A: track 34.7 -> 30.7 mm
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