File: PCB/Aida_Base/Aida_Base.kicad_pcb (KiCad board)
At the start: 2 copper layers, 242.9 x 83.3 mm, 228 parts, among them J1 AudioJack4, J10 Conn_01x03_Pin, J11 Conn_01x04_Pin, J12 Conn_01x04_Pin, J13 Conn_01x04_Pin, J14 Conn_01x04_Pin, J15 Conn_01x04_Pin, J16 Conn_01x04_Pin, J17 Conn_02x02_Odd_Even, J18 Conn_02x02_Odd_Even, J19 Conn_01x04_Pin, J2 AudioJack4, J20 Conn_01x06_Pin, J21 Conn_01x06_Pin, J22 Conn_01x04_Pin, J23 Conn_01x02_Pin, J24 Conn_01x02_Pin, J3 USB_C_Receptacle_L, J4 USB_C_Receptacle_R, J5 Conn_01x02_Pin, J6 Conn_01x02_Pin, J7 Conn_01x05_Pin, J8 Conn_01x05_Pin, J9 Conn_01x03_Pin, Q1 BSS138, Q2 BSS138, SW1 Boot, SW2 BOOT, SW3 RESET, SW4 RESET, U3 RP2040_L, U4 RP2040_R, U5 W25Q128JVS, U6 W25Q128JVS, U7 AP2112K-3.3, U8 AP2112K-3.3, Y1 12MHz, Y2 12MHz

Commit message: LEDのフットプリント変更。配線調整中。
Parts:
- L1, L2, L3, L4, L5, L6: footprint Lib_Local:YS-SK6812MINI-E_middle_hole_with_small_pad -> Lib_Local:YS-SK6812MINI-E_middle_hole_with_small_pad_NPTH
Routing:
- net +3V3_L: track 208.9 -> 204.2 mm, vias 9 -> 10
- net RESET_L: track 66.8 -> 69.7 mm
- net SCL_L: track 82.3 -> 80.2 mm
- net SDA_L: track 84.4 -> 82.8 mm
- net ROW_L_1: track 160.9 -> 159.3 mm
- net USB_BOOT_L: track 72.9 -> 71.5 mm
- net ENC_L_A: track 31.2 -> 32.0 mm
- net COL_L_5: track 120.8 -> 120.1 mm
- net SWDIO_L: track 70.2 -> 69.7 mm
- net SWCLK_L: track 74.2 -> 73.7 mm

Commit message: 配線調整
Parts:
- SW2: value BOOT -> Boot
- SW3, SW4: value RESET -> Reset
Routing:
- net ROW_R_0: track 151.5 -> 161.2 mm, vias 6 -> 7
- net COL_R_5: track 114.2 -> 120.1 mm
- net COL_R_4: track 134.2 -> 139.3 mm
- net SWDIO_R: track 63.9 -> 60.2 mm
- net +3V3_R: track 246.6 -> 243.0 mm
- net COL_R_2: track 109.8 -> 106.6 mm
- net GND_R: track 30.9 -> 33.9 mm, vias 35 -> 44
- net ROW_R_3: track 169.5 -> 172.3 mm
- net COL_R_3: track 119.8 -> 117.9 mm, vias 5 -> 4
- net COL_R_1: track 129.9 -> 128.3 mm
- net SWCLK_R: track 67.3 -> 65.9 mm
- net RESET_R: track 80.2 -> 78.8 mm
- net COL_L_2: track 131.2 -> 132.5 mm
- net ROW_R_2: track 124.1 -> 125.4 mm
- net SDA_R: track 65.6 -> 64.5 mm
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
Commit message: USB配線長を調整した
Routing:
- net D_R-: track 75.4 -> 76.4 mm
- net +5V_R: track 156.4 -> 155.9 mm
- net GND_R: track 33.9 -> 34.1 mm, vias 44 -> 59
- net GND_L: vias 58 -> 75

Commit message: 開発ナンバーと表裏を記載
Other:
- board text added: "Aida DN0010 by @jpskenn"
- board text added: "L Back"
- board text added: "R Back"
Changed lines of the file:
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@@
 		(layer "User.1")
+	)
+	(gr_text "Aida DN0010\nby @jpskenn"
+		(at 57.15 58.340625 0)
+		(layer "B.SilkS")
+		(effects
+			(font
+				(size 1 1)
+				(thickness 0.1)
+			)
+			(justify left bottom mirror)
+		)
+	)
+	(gr_text "L Back"
+		(at 78.58125 38.1 0)
+		(layer "B.SilkS" knockout)
+		(effects
+			(font
+				(size 3 3)
+				(thickness 0.375)
+				(italic yes)
+			)
+			(justify left bottom mirror)
+		)
+	)
+	(gr_text "R Back"
+		(at 242.8875 38.1 0)
+		(layer "B.SilkS" knockout)
+		(effects
+			(font
+				(size 3 3)
+				(thickness 0.375)
+				(italic yes)
+			)
+			(justify left bottom mirror)
+		)
+	)
+	(gr_text "Aida DN0010\nby @jpskenn"
+		(at 257.175 58.340625 0)
+		(layer "B.SilkS")
+		(effects
+			(font
+				(size 1 1)
+				(thickness 0.1)
+			)
+			(justify left bottom mirror)
+		)
 	)
 	(gr_text "Top PCB outline"
