File: PCB/Aida_Base/Aida_Base.kicad_sch (KiCad schematic)
At the start: 232 parts, among them J1 AudioJack4, J10 Conn_01x03_Pin, J11 Conn_01x04_Pin, J12 Conn_01x04_Pin, J13 Conn_01x04_Pin, J14 Conn_01x04_Pin, J15 Conn_01x04_Pin, J16 Conn_01x04_Pin, J17 Conn_02x02_Odd_Even, J18 Conn_02x02_Odd_Even, J19 Conn_01x04_Pin, J2 AudioJack4, J20 Conn_01x06_Pin, J21 Conn_01x06_Pin, J22 Conn_01x04_Pin, J23 Conn_01x02_Pin, J24 Conn_01x02_Pin, J3 USB_C_Receptacle_L, J4 USB_C_Receptacle_R, J5 Conn_01x02_Pin, J6 Conn_01x02_Pin, J7 Conn_01x05_Pin, J8 Conn_01x05_Pin, J9 Conn_01x03_Pin, Q1 BSS138, Q2 BSS138, SW1 Boot, SW2 Boot, SW3 Reset, SW4 Reset, U3 RP2040_L, U4 RP2040_R, U5 W25Q128JVS, U6 W25Q128JVS, U7 AP2112K-3.3, U8 AP2112K-3.3, Y1 12MHz, Y2 12MHz

Commit message: スルーホールタップの型番変更に伴い、ランド、3Dモデルも変更。
Parts:
- H1, H11, H12, H13, H14, H15, H16, H17, H18, H19, H2, H20, H3, H4, H5, H6, H7, H8: footprint Lib_Local:MountingHole_M2_Through-hole_tap_THC-0.8-2.0-2_minimal -> Lib_Local:MountingHole_M2_Through-hole_tap_TH-0.8-2.0-M2_minimal
- H_btm_L3, H_btm_L4, H_btm_L5, H_btm_L6, H_btm_R3, H_btm_R4, H_btm_R5, H_btm_R6: footprint Lib_Local:MountingHole_M2_Through-hole_tap_THC-0.8-1.0-2_minimal -> Lib_Local:MountingHole_M2_Through-hole_tap_TH-0.8-1.0-M2_minimal
- H_mid_L1, H_mid_L2, H_mid_R1, H_mid_R2: footprint Lib_Local:MountingHole_M2_Through-hole_tap_THC-0.8-1.0-2_minimal -> Lib_Local:MountingHole_M2_Through-hole_tap_TH-0.8-2.0-M2_minimal
Changed lines of the file:
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@@
 			)
 		)
-		(property "Footprint" "Lib_Local:MountingHole_M2_Through-hole_tap_THC-0.8-2.0-2_minimal"
+		(property "Footprint" "Lib_Local:MountingHole_M2_Through-hole_tap_TH-0.8-2.0-M2_minimal"
 			(at 186.69 62.23 0)
 			(effects
@@
 			)
 		)
-		(property "Footprint" "Lib_Local:MountingHole_M2_Through-hole_tap_THC-0.8-2.0-2_minimal"
+		(property "Footprint" "Lib_Local:MountingHole_M2_Through-hole_tap_TH-0.8-2.0-M2_minimal"
 			(at 161.29 36.83 0)
 			(effects
@@
 			)
 		)
-		(property "Footprint" "Lib_Local:MountingHole_M2_Through-hole_tap_THC-0.8-2.0-2_minimal"
+		(property "Footprint" "Lib_Local:MountingHole_M2_Through-hole_tap_TH-0.8-2.0-M2_minimal"
 			(at 168.91 53.34 0)
 			(effects
@@
 			)
 		)
-		(property "Footprint" "Lib_Local:MountingHole_M2_Through-hole_tap_THC-0.8-2.0-2_minimal"
+		(property "Footprint" "Lib_Local:MountingHole_M2_Through-hole_tap_TH-0.8-2.0-M2_minimal"
 			(at 340.36 36.83 0)
 			(effects
@@
 			)
 		)
-		(property "Footprint" "Lib_Local:MountingHole_M2_Through-hole_tap_THC-0.8-2.0-2_minimal"
+		(property "Footprint" "Lib_Local:MountingHole_M2_Through-hole_tap_TH-0.8-2.0-M2_minimal"
 			(at 118.11 40.64 0)
 			(effects
@@
 			)
 		)
-		(property "Footprint" "Lib_Local:MountingHole_M2_Through-hole_tap_THC-0.8-2.0-2_minimal"
+		(property "Footprint" "Lib_Local:MountingHole_M2_Through-hole_tap_TH-0.8-2.0-M2_minimal"
 			(at 335.28 53.34 0)
 			(effects
@@
 			)
 		)
-		(property "Footprint" "Lib_Local:MountingHole_M2_Through-hole_tap_THC-0.8-2.0-2_minimal"
+		(property "Footprint" "Lib_Local:MountingHole_M2_Through-hole_tap_TH-0.8-2.0-M2_minimal"
 			(at 322.58 66.04 0)
 			(effects
@@
 			)
 		)
-		(property "Footprint" "Lib_Local:MountingHole_M2_Through-hole_tap_THC-0.8-1.0-2_minimal"
+		(property "Footprint" "Lib_Local:MountingHole_M2_Through-hole_tap_TH-0.8-1.0-M2_minimal"
 			(at 214.63 275.59 0)
 			(effects
@@
 			)
 		)
-		(property "Footprint" "Lib_Local:MountingHole_M2_Through-hole_tap_THC-0.8-2.0-2_minimal"
+		(property "Footprint" "Lib_Local:MountingHole_M2_Through-hole_tap_TH-0.8-2.0-M2_minimal"
 			(at 386.08 40.64 0)
 			(effects
@@
 			)
 		)
-		(property "Footprint" "Lib_Local:MountingHole_M2_Through-hole_tap_THC-0.8-1.0-2_minimal"
+		(property "Footprint" "Lib_Local:MountingHole_M2_Through-hole_tap_TH-0.8-2.0-M2_minimal"
 			(at 71.12 266.7 0)
 			(effects
@@
 			)
 		)
-		(property "Footprint" "Lib_Local:MountingHole_M2_Through-hole_tap_THC-0.8-1.0-2_minimal"
+		(property "Footprint" "Lib_Local:MountingHole_M2_Through-hole_tap_TH-0.8-1.0-M2_minimal"
 			(at 39.37 275.59 0)
 			(effects
@@
 			)
 		)
-		(property "Footprint" "Lib_Local:MountingHole_M2_Through-hole_tap_THC-0.8-2.0-2_minimal"
+		(property "Footprint" "Lib_Local:MountingHole_M2_Through-hole_tap_TH-0.8-2.0-M2_minimal"
 			(at 340.36 49.53 0)
 			(effects
@@
 			)
 		)
-		(property "Footprint" "Lib_Local:MountingHole_M2_Through-hole_tap_THC-0.8-2.0-2_minimal"
+		(property "Footprint" "Lib_Local:MountingHole_M2_Through-hole_tap_TH-0.8-2.0-M2_minimal"
 			(at 173.99 36.83 0)
 			(effects
@@
 			)
 		)
-		(property "Footprint" "Lib_Local:MountingHole_M2_Through-hole_tap_THC-0.8-2.0-2_minimal"
+		(property "Footprint" "Lib_Local:MountingHole_M2_Through-hole_tap_TH-0.8-2.0-M2_minimal"
 			(at 391.16 36.83 0)
 			(effects
@@
 			)
 		)
-		(property "Footprint" "Lib_Local:MountingHole_M2_Through-hole_tap_THC-0.8-2.0-2_minimal"
+		(property "Footprint" "Lib_Local:MountingHole_M2_Through-hole_tap_TH-0.8-2.0-M2_minimal"
 			(at 156.21 40.64 0)
 			(effects
@@
 			)
 		)
-		(property "Footprint" "Lib_Local:MountingHole_M2_Through-hole_tap_THC-0.8-1.0-2_minimal"
+		(property "Footprint" "Lib_Local:MountingHole_M2_Through-hole_tap_TH-0.8-1.0-M2_minimal"
 			(at 19.05 270.51 0)
 			(effects
@@
 			)
 		)
-		(property "Footprint" "Lib_Local:MountingHole_M2_Through-hole_tap_THC-0.8-2.0-2_minimal"
+		(property "Footprint" "Lib_Local:MountingHole_M2_Through-hole_tap_TH-0.8-2.0-M2_minimal"
 			(at 327.66 62.23 0)
 			(effects
@@
 			)
 		)
-		(property "Footprint" "Lib_Local:MountingHole_M2_Through-hole_tap_THC-0.8-1.0-2_minimal"
+		(property "Footprint" "Lib_Local:MountingHole_M2_Through-hole_tap_TH-0.8-2.0-M2_minimal"
 			(at 269.24 266.7 0)
 			(effects
@@
 			)
 		)
-		(property "Footprint" "Lib_Local:MountingHole_M2_Through-hole_tap_THC-0.8-1.0-2_minimal"
+		(property "Footprint" "Lib_Local:MountingHole_M2_Through-hole_tap_TH-0.8-1.0-M2_minimal"
 			(at 16.51 275.59 0)
 			(effects
@@
 			)
 		)
-		(property "Footprint" "Lib_Local:MountingHole_M2_Through-hole_tap_THC-0.8-2.0-2_minimal"
+		(property "Footprint" "Lib_Local:MountingHole_M2_Through-hole_tap_TH-0.8-2.0-M2_minimal"
 			(at 347.98 40.64 0)
 			(effects
@@
 			)
 		)
-		(property "Footprint" "Lib_Local:MountingHole_M2_Through-hole_tap_THC-0.8-2.0-2_minimal"
+		(property "Footprint" "Lib_Local:MountingHole_M2_Through-hole_tap_TH-0.8-2.0-M2_minimal"
 			(at 123.19 36.83 0)
 			(effects
@@
 			)
 		)
-		(property "Footprint" "Lib_Local:MountingHole_M2_Through-hole_tap_THC-0.8-2.0-2_minimal"
+		(property "Footprint" "Lib_Local:MountingHole_M2_Through-hole_tap_TH-0.8-2.0-M2_minimal"
 			(at 181.61 66.04 0)
 			(effects
@@
 			)
 		)
-		(property "Footprint" "Lib_Local:MountingHole_M2_Through-hole_tap_THC-0.8-1.0-2_minimal"
+		(property "Footprint" "Lib_Local:MountingHole_M2_Through-hole_tap_TH-0.8-1.0-M2_minimal"
 			(at 234.95 270.51 0)
 			(effects
@@
 			)
 		)
-		(property "Footprint" "Lib_Local:MountingHole_M2_Through-hole_tap_THC-0.8-1.0-2_minimal"
+		(property "Footprint" "Lib_Local:MountingHole_M2_Through-hole_tap_TH-0.8-1.0-M2_minimal"
 			(at 237.49 275.59 0)
 			(effects
@@
 			)
 		)
-		(property "Footprint" "Lib_Local:MountingHole_M2_Through-hole_tap_THC-0.8-1.0-2_minimal"
+		(property "Footprint" "Lib_Local:MountingHole_M2_Through-hole_tap_TH-0.8-2.0-M2_minimal"
 			(at 87.63 266.7 0)
 			(effects
@@
 			)
 		)
-		(property "Footprint" "Lib_Local:MountingHole_M2_Through-hole_tap_THC-0.8-2.0-2_minimal"
+		(property "Footprint" "Lib_Local:MountingHole_M2_Through-hole_tap_TH-0.8-2.0-M2_minimal"
 			(at 353.06 36.83 0)
 			(effects
@@
 			)
 		)
-		(property "Footprint" "Lib_Local:MountingHole_M2_Through-hole_tap_THC-0.8-1.0-2_minimal"
+		(property "Footprint" "Lib_Local:MountingHole_M2_Through-hole_tap_TH-0.8-1.0-M2_minimal"
 			(at 36.83 270.51 0)
 			(effects
@@
 			)
 		)
-		(property "Footprint" "Lib_Local:MountingHole_M2_Through-hole_tap_THC-0.8-1.0-2_minimal"
+		(property "Footprint" "Lib_Local:MountingHole_M2_Through-hole_tap_TH-0.8-2.0-M2_minimal"
 			(at 285.75 266.7 0)
 			(effects
@@
 			)
 		)
-		(property "Footprint" "Lib_Local:MountingHole_M2_Through-hole_tap_THC-0.8-2.0-2_minimal"
+		(property "Footprint" "Lib_Local:MountingHole_M2_Through-hole_tap_TH-0.8-2.0-M2_minimal"
 			(at 173.99 49.53 0)
 			(effects
@@
 			)
 		)
-		(property "Footprint" "Lib_Local:MountingHole_M2_Through-hole_tap_THC-0.8-1.0-2_minimal"
+		(property "Footprint" "Lib_Local:MountingHole_M2_Through-hole_tap_TH-0.8-1.0-M2_minimal"
 			(at 217.17 270.51 0)
 			(effects

Commit message: BOM記入
Parts:
- C10, C11, C12, C13, C14, C15, C16, C17, C18, C19, C20, C22, C23, C25, C26, C5, C6, C7, C8, C9: LCSC (none) -> C1525
- C27, C28, C29, C30: LCSC (none) -> C52923
- C31, C35: LCSC C1525 -> C23733
- D43, D44: LCSC C78442 -> C558444
- D45, D46: LCSC (none) -> C81598
- H_mid_L1, H_mid_L2, H_mid_R1, H_mid_R2, J10, J11, J12, J13, J14, J15, J16, J17, J18, J19, J20, J21, J22, J23, J24, J5, J6, J7, J8, J9, SW_RE_L1, SW_RE_L2, TP1, TP2: now left out of the parts list
- J1, J2: LCSC (none) -> C18185602
- J3, J4: LCSC (none) -> C165948
- L1, L2, L3, L4, L5, L6: LCSC (none) -> C5149201
- LS1, LS2: LCSC (none) -> C910763
- R1, R15, R17, R2, R21, R22: LCSC (none) -> C11702
- R16, R18, R3, R4: LCSC (none) -> C25104
- R19, R20: LCSC (none) -> C25744
- R23, R24, R25, R26: LCSC (none) -> C25900
- R27, R28, R29, R30: LCSC (none) -> C25100
- R5, R6, R7, R8: LCSC (none) -> C25905
- STLED1, STLED2: LCSC (none) -> C130723
- U3, U4: LCSC (none) -> C2040
- U5, U6: LCSC (none) -> C190862
- U7, U8: LCSC (none) -> C51118
- Y1, Y2: LCSC (none) -> C341520
