File: PCB/Aida_Mid_Outside/Aida_Mid_Outside.kicad_pcb (KiCad board)
At the start: 2 copper layers, 25.7 x 23.5 mm, 6 parts

Commit message: テストポイントを追加、配置した。
Parts:
- added TP1: COL0_from, Connector_PinHeader_2.00mm:PinHeader_1x01_P2.00mm_Vertical, F.Cu at (45.8, 39.9)
- added TP2: COL0_to, Connector_PinHeader_2.00mm:PinHeader_1x01_P2.00mm_Vertical, F.Cu at (44.1, 47.6)
- added TP3: GND, Connector_PinHeader_2.00mm:PinHeader_1x01_P2.00mm_Vertical, F.Cu at (53.6, 36.3)
Routing:
- net COL_0_from_Base: track 20.9 -> 25.7 mm
- net COL_0_to_Base: track 23.6 -> 27.4 mm

Commit message: 原点ガイドを追加。基板Mid_InsideのLED穴形状調整
Other:
- board text added: "Center Origin"
- board text added: "Grid Origin"
Changed lines of the file:
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@@
 		(layer "Edge.Cuts")
+	)
+	(gr_line
+		(start 23.8125 21.43125)
+		(end 23.8125 26.19375)
+		(stroke
+			(width 0.1)
+			(type default)
+		)
+		(layer "User.1")
+	)
+	(gr_line
+		(start 152.4 21.43125)
+		(end 152.4 26.19375)
+		(stroke
+			(width 0.1)
+			(type default)
+		)
+		(layer "User.1")
+	)
+	(gr_line
+		(start 21.43125 23.8125)
+		(end 26.19375 23.8125)
+		(stroke
+			(width 0.1)
+			(type default)
+		)
+		(layer "User.1")
+	)
+	(gr_circle
+		(center 152.4 23.8125)
+		(end 153.590625 23.8125)
+		(stroke
+			(width 0.1)
+			(type default)
+		)
+		(fill no)
+		(layer "User.1")
+	)
+	(gr_line
+		(start 150.01875 23.8125)
+		(end 154.78125 23.8125)
+		(stroke
+			(width 0.1)
+			(type default)
+		)
+		(layer "User.1")
+	)
+	(gr_circle
+		(center 23.8125 23.8125)
+		(end 25.003125 23.8125)
+		(stroke
+			(width 0.1)
+			(type default)
+		)
+		(fill no)
+		(layer "User.1")
 	)
 	(gr_text "PCB Mid-Outside outline"
@@
 		)
 	)
+	(gr_text "Grid Origin"
+		(at 20.240625 21.43125 0)
+		(layer "User.1")
+		(effects
+			(font
+				(size 1 1)
+				(thickness 0.15)
+			)
+			(justify left bottom)
+		)
+	)
+	(gr_text "Center Origin"
+		(at 148.828125 21.43125 0)
+		(layer "User.1")
+		(effects
+			(font
+				(size 1 1)
+				(thickness 0.15)
+			)
+			(justify left bottom)
+		)
+	)
 	(segment
 		(start 42.267203 42.862516)
@@
 		)
 	)
+	(group ""
+		(members "2517ec00-a1db-4c22-ba1d-3de02ac446b4" "270d3d59-ed5c-49c9-bb77-50ed0e8d9958"
+			"6fc48c44-e3b3-4c31-a620-ada293b59cd9" "deab2e9b-347a-4123-a799-33c7d25d06d1"
+		)
+	)
+	(group ""
+		(members "3f858eb7-bc97-4a22-90a0-ebcbffb16d23" "89fb3b80-6500-4d71-832e-93b456a59019"
+			"960ad950-f809-49cc-a18b-b68c7fa7d76f" "c8bab62e-eccd-4a95-bcaf-3c1ffeaf97d6"
+		)
+	)

Commit message: 開発ナンバーと表裏を記載
Other:
- board text added: "Aida DN0010 by @jpskenn"
- board text added: "L Back"
- board text added: "R Back"
Changed lines of the file:
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@@
 		(layer "User.1")
+	)
+	(gr_text "R Back"
+		(at 41.67189 38.100012 0)
+		(layer "F.SilkS" knockout)
+		(effects
+			(font
+				(size 1.8 1.8)
+				(thickness 0.225)
+				(italic yes)
+			)
+			(justify left bottom)
+		)
+	)
+	(gr_text "Aida DN0010\nby @jpskenn"
+		(at 57.150028 41.67189 0)
+		(layer "B.SilkS")
+		(effects
+			(font
+				(size 1 1)
+				(thickness 0.1)
+			)
+			(justify left bottom mirror)
+		)
+	)
+	(gr_text "L Back"
+		(at 51.792211 38.100012 0)
+		(layer "B.SilkS" knockout)
+		(effects
+			(font
+				(size 1.8 1.8)
+				(thickness 0.225)
+				(italic yes)
+			)
+			(justify left bottom mirror)
+		)
 	)
 	(gr_text "PCB Mid-Outside outline"
