File: PCB/Aida_Plate_Mid_Outside/Aida_Plate_Mid_Outside.kicad_pcb (KiCad board)
At the start: 2 copper layers, 25.7 x 23.5 mm, 4 parts

Commit message: 原点ガイドを追加。基板Mid_InsideのLED穴形状調整
Other:
- board text added: "Center Origin"
- board text added: "Grid Origin"
Changed lines of the file:
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@@
 		(layer "Edge.Cuts")
+	)
+	(gr_circle
+		(center 152.4 23.8125)
+		(end 153.590625 23.8125)
+		(stroke
+			(width 0.1)
+			(type default)
+		)
+		(fill no)
+		(layer "User.1")
+	)
+	(gr_line
+		(start 23.8125 21.43125)
+		(end 23.8125 26.19375)
+		(stroke
+			(width 0.1)
+			(type default)
+		)
+		(layer "User.1")
+	)
+	(gr_line
+		(start 150.01875 23.8125)
+		(end 154.78125 23.8125)
+		(stroke
+			(width 0.1)
+			(type default)
+		)
+		(layer "User.1")
+	)
+	(gr_circle
+		(center 23.8125 23.8125)
+		(end 25.003125 23.8125)
+		(stroke
+			(width 0.1)
+			(type default)
+		)
+		(fill no)
+		(layer "User.1")
+	)
+	(gr_line
+		(start 21.43125 23.8125)
+		(end 26.19375 23.8125)
+		(stroke
+			(width 0.1)
+			(type default)
+		)
+		(layer "User.1")
+	)
+	(gr_line
+		(start 152.4 21.43125)
+		(end 152.4 26.19375)
+		(stroke
+			(width 0.1)
+			(type default)
+		)
+		(layer "User.1")
 	)
 	(gr_text "PCB Mid-Outside outline"
 		(at 0.595293 41.076577 0)
 		(layer "Eco2.User")
+		(effects
+			(font
+				(size 1 1)
+				(thickness 0.15)
+			)
+			(justify left bottom)
+		)
+	)
+	(gr_text "Center Origin"
+		(at 148.828125 21.43125 0)
+		(layer "User.1")
+		(effects
+			(font
+				(size 1 1)
+				(thickness 0.15)
+			)
+			(justify left bottom)
+		)
+	)
+	(gr_text "Grid Origin"
+		(at 20.240625 21.43125 0)
+		(layer "User.1")
 		(effects
 			(font
@@
 		)
 	)
+	(group ""
+		(members "169248b9-887c-4371-bec6-2f7670015c0d" "77dab541-745d-4d72-a772-946c405ac248"
+			"8c8e3d5d-f474-49e6-bcbb-f4b597831ad7" "f9786ac8-6e7b-4a39-8dcf-4a2f092b66c8"
+		)
+	)
+	(group ""
+		(members "2c8ee198-8e25-4875-971a-ee7228c78479" "930981f7-af5a-4b44-a047-11e674e6b797"
+			"a2620f69-a36b-4687-bc1a-0be638fadd87" "dae946b0-d9f2-4f8b-975d-fac624484f86"
+		)
+	)
