File: PCB/Aida_Plate_Top/Aida_Plate_Top.kicad_pcb (KiCad board)
At the start: 2 copper layers, 31 x 23.5 mm, 4 parts

Commit message: 原点ガイドを追加。基板Mid_InsideのLED穴形状調整
Other:
- board text added: "Center Origin"
- board text added: "Grid Origin"
Changed lines of the file:
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@@
 		(layer "Edge.Cuts")
+	)
+	(gr_circle
+		(center 23.8125 23.8125)
+		(end 25.003125 23.8125)
+		(stroke
+			(width 0.1)
+			(type default)
+		)
+		(fill no)
+		(layer "User.1")
+	)
+	(gr_line
+		(start 23.8125 21.43125)
+		(end 23.8125 26.19375)
+		(stroke
+			(width 0.1)
+			(type default)
+		)
+		(layer "User.1")
+	)
+	(gr_circle
+		(center 152.4 23.8125)
+		(end 153.590625 23.8125)
+		(stroke
+			(width 0.1)
+			(type default)
+		)
+		(fill no)
+		(layer "User.1")
+	)
+	(gr_line
+		(start 150.01875 23.8125)
+		(end 154.78125 23.8125)
+		(stroke
+			(width 0.1)
+			(type default)
+		)
+		(layer "User.1")
+	)
+	(gr_line
+		(start 152.4 21.43125)
+		(end 152.4 26.19375)
+		(stroke
+			(width 0.1)
+			(type default)
+		)
+		(layer "User.1")
+	)
+	(gr_line
+		(start 21.43125 23.8125)
+		(end 26.19375 23.8125)
+		(stroke
+			(width 0.1)
+			(type default)
+		)
+		(layer "User.1")
 	)
 	(gr_text "Top PCB outline"
 		(at 119.657906 32.444558 0)
 		(layer "Eco1.User")
+		(effects
+			(font
+				(size 1 1)
+				(thickness 0.15)
+			)
+			(justify left bottom)
+		)
+	)
+	(gr_text "Grid Origin"
+		(at 20.240625 21.43125 0)
+		(layer "User.1")
+		(effects
+			(font
+				(size 1 1)
+				(thickness 0.15)
+			)
+			(justify left bottom)
+		)
+	)
+	(gr_text "Center Origin"
+		(at 148.828125 21.43125 0)
+		(layer "User.1")
 		(effects
 			(font
@@
 		)
 	)
+	(group ""
+		(members "65a8c0aa-0671-4e80-8228-1b390929ce33" "9ef5eefa-8089-4df9-9158-13d259b78a8e"
+			"c6f8489c-a328-48ae-af65-e3d4a1b4307a" "eb766416-8578-464a-9db3-896550ced98a"
+		)
+	)
+	(group ""
+		(members "0f4e376c-d207-45e9-a339-4a1034974593" "16bcb8a0-e2db-42b9-87ec-a259e6635806"
+			"1c97c020-069d-4a5c-a890-91756e4b4f1c" "fae46e53-90d6-49c5-b29b-1034657bdb79"
+		)
+	)
